Commit message: Add initial Franka Desk Stuff

File: franka_fer_moveit_config/srdf/fer_arm_hand.xacro (robot description, xacro)
@@ -1,5 +1,5 @@
 <?xml version='1.0' encoding='utf-8'?>
-<robot xmlns:xacro="http://www.ros.org/wiki/xacro" name="fr3">
-  <xacro:macro name="fr3_arm_hand" params="arm_id:='fr3' ">
+<robot xmlns:xacro="http://www.ros.org/wiki/xacro" name="fer">
+  <xacro:macro name="fer_arm_hand" params="arm_id:='fer' ">
     <group_state name="open" group="hand">
       <joint name="${arm_id}_finger_joint1" value="0.035"/>

File: franka_fer_moveit_config/srdf/group_definition.xacro (robot description, xacro)
@@ -1,4 +1,4 @@
 <?xml version="1.0" encoding="UTF-8"?>
-<robot xmlns:xacro="http://www.ros.org/wiki/xacro" name="fr3">
+<robot xmlns:xacro="http://www.ros.org/wiki/xacro" name="fer">
   <xacro:macro name="group_definition" params="group_name arm_id tip_link">
     <group name="${group_name}">

Commit message: Updated Desktop Client

File: franka_fer_moveit_config/srdf/fer_arm_hand.xacro (robot description, xacro)
@@ -3,6 +3,6 @@
   <xacro:macro name="fer_arm_hand" params="arm_id:='fer' ">
     <group_state name="open" group="hand">
-      <joint name="${arm_id}_finger_joint1" value="0.035"/>
-      <joint name="${arm_id}_finger_joint2" value="0.035"/>
+      <joint name="${arm_id}_finger_joint1" value="0.026"/>
+      <joint name="${arm_id}_finger_joint2" value="0.026"/>
     </group_state>
     <group_state name="close" group="hand">
